Commit message: tried to add sensor

File: kinova_description/urdf/arm_on_table.xacro (robot description, xacro)
@@ -47,3 +47,22 @@
 		<child link="root"/>
 	</joint>
+	<!-- Add the Xtion to the table to observe the real arm: code from here https://github.com/JenniferBuehler/common-sensors.git
+	<joint name="toxtion_base" type="fixed">
+        <origin xyz="0 0 0.1" rpy="0 0 -1.57079632679" />
+        <parent link="j2n6s300_link_6" />
+        <child link="xtion_base" />
+    </joint>
+    <link name="xtion_base">
+        <visual>
+            <origin xyz="0 0 0" rpy="0 0 0" />
+            <geometry>
+                <box size="0 0 0"/>
+            </geometry>
+            <material name="orange"/>
+        </visual>
+    </link>
+    <xacro:include filename="$(find common_sensors)/urdf/sensors/xtion.urdf.xacro"/>>
+    <xacro:sensor_xtion parent="xtion_base" camera_name="xtion">
+		<origin xyz="0 0 0" rpy="0 0 0" />
+	</xacro:sensor_xtion>  -->
 </robot>

File: kinova_description/urdf/objects/arm_stand.xacro (robot description, xacro)
@@ -1,3 +1,2 @@
- <!-- All code for the table is taking from https://github.com/JenniferBuehler/jaco-arm-pkgs -->
 <?xml version="1.0" encoding="UTF-8"?>
 <root xmlns:xacro="http://ros.org/wiki/xacro">

File: kinova_description/urdf/objects/table.xacro (robot description, xacro)
@@ -1,11 +1,10 @@
- <!-- All code for the table is taking from https://github.com/JenniferBuehler/jaco-arm-pkgs -->
 <?xml version="1.0" encoding="UTF-8"?>
 <root xmlns:xacro="http://ros.org/wiki/xacro">
     <xacro:macro name="default_material">
-	<mu1>0.9</mu1>
-	<mu2>0.9</mu2>
-    	<kp>1000000.0</kp>
-    	<kd>1.0</kd>
-	<dynamics damping="0.7" friction="100.0" />
+    <mu1>0.9</mu1>
+    <mu2>0.9</mu2>
+        <kp>1000000.0</kp>
+        <kd>1.0</kd>
+    <dynamics damping="0.7" friction="100.0" />
     </xacro:macro>
     <gazebo reference="table_base">

Commit message: paused gazebo to prevent collision

File: kinova_description/urdf/arm_on_table.xacro (robot description, xacro)
@@ -39,7 +39,4 @@
 		</collision>
 	</link>
-	<property name="robot_root" value="root" />
-	<xacro:include filename="$(find kinova_description)/urdf/j2n6s300.xacro"/>
-	<xacro:j2n6s300 base_parent="${robot_root}"/>
 	<joint name="jaco_to_table" type="fixed">
 		<origin xyz="-0.000482247085224208 0.08 -0.000503436190578577" rpy="1.57079632679 0 3.14159265359" />
@@ -47,22 +44,20 @@
 		<child link="root"/>
 	</joint>
-	<!-- Add the Xtion to the table to observe the real arm: code from here https://github.com/JenniferBuehler/common-sensors.git
+	<!-- Add robot arm -->
+	<property name="robot_root" value="root" />
+	<xacro:include filename="$(find kinova_description)/urdf/j2n6s300.xacro"/>
+	<xacro:j2n6s300 base_parent="${robot_root}"/>
+	<!-- Add the Xtion to the table to observe the real arm: code from here https://github.com/JenniferBuehler/common-sensors.git -->
 	<joint name="toxtion_base" type="fixed">
-        <origin xyz="0 0 0.1" rpy="0 0 -1.57079632679" />
-        <parent link="j2n6s300_link_6" />
+        <origin xyz="0 -0.89 -0.01" rpy="0 0 0" />
+        <parent link="tabletop_corner" />
         <child link="xtion_base" />
     </joint>
     <link name="xtion_base">
-        <visual>
-            <origin xyz="0 0 0" rpy="0 0 0" />
-            <geometry>
-                <box size="0 0 0"/>
-            </geometry>
-            <material name="orange"/>
-        </visual>
+        <static>false</static>
     </link>
     <xacro:include filename="$(find common_sensors)/urdf/sensors/xtion.urdf.xacro"/>>
     <xacro:sensor_xtion parent="xtion_base" camera_name="xtion">
-		<origin xyz="0 0 0" rpy="0 0 0" />
-	</xacro:sensor_xtion>  -->
+		<origin xyz="0 0 1" rpy="0 -1.57079632679 -1.57079632679" />
+	</xacro:sensor_xtion>
 </robot>

File: kinova_description/urdf/objects/arm_stand.xacro (robot description, xacro)
@@ -23,5 +23,6 @@
                 <origin xyz="0 0 0" rpy="0 0 0" />
                 <geometry>
-                    <mesh filename="package://kinova_description/meshes/objects/arm_stand.STL" />
+                    <box size = "0 0 0"/>
+                    <!-- <mesh filename="package://kinova_description/meshes/objects/arm_stand.STL" /> -->
                 </geometry>
             </collision>

Commit message: figure out home position

File: kinova_description/urdf/arm_on_table.xacro (robot description, xacro)
@@ -3,4 +3,5 @@
 <robot name="j2n6s300_on_table" xmlns:xacro="http://ros.org/wiki/xacro">
 	<link name="world"/>
+	<xacro:include filename="$(find kinova_description)/urdf/j2n6s300.xacro"/>
 	<joint name="base_to_jaco_on_table" type="fixed">
 		<origin xyz="0 0 0" rpy="0 0 0" />
@@ -13,5 +14,5 @@
 	<xacro:include filename="$(find kinova_description)/urdf/objects/table.xacro" />
 	<joint name="table_to_arm" type="fixed">
-		<origin xyz="0.40488474042 0.27988474042 0.3" rpy="0 0 -0.785398163397458" />
+		<origin xyz="0.40488474042 0.27988474042 0.3" rpy="0 0 -${J_PI/4}" />
 		<parent link="robot_base"/>
 		<child link="table_base"/>
@@ -20,5 +21,5 @@
 	<xacro:arm_stand_link link_name="arm_stand"/>
 	<joint name="j2b" type="fixed">
-		<origin xyz="0 -0.035 0" rpy="-1.57079632679 -3.14159265358979 0" /> <!-- set the arm "inside" the table for now because of the rim along the real table. creating a bit of a buffer zone so moveit trajectories are within safe distance of the table edges. -->
+		<origin xyz="0 -0.035 0" rpy="-${J_PI/2} -${J_PI} 0" /> <!-- set the arm "inside" the table for now because of the rim along the real table. creating a bit of a buffer zone so moveit trajectories are within safe distance of the table edges. -->
 		<parent link="tabletop_corner" />
 		<child link="arm_stand" />
@@ -40,5 +41,5 @@
 	</link>
 	<joint name="jaco_to_table" type="fixed">
-		<origin xyz="-0.000482247085224208 0.08 -0.000503436190578577" rpy="1.57079632679 0 3.14159265359" />
+		<origin xyz="-0.000482247085224208 0.08 -0.000503436190578577" rpy="${J_PI/2} 0 ${J_PI}" />
 		<parent link="arm_stand"/>
 		<child link="root"/>
@@ -46,10 +47,9 @@
 	<!-- Add robot arm -->
 	<property name="robot_root" value="root" />
-	<xacro:include filename="$(find kinova_description)/urdf/j2n6s300.xacro"/>
 	<xacro:j2n6s300 base_parent="${robot_root}"/>
-	<!-- Add the Xtion to the table to observe the real arm: code from here https://github.com/JenniferBuehler/common-sensors.git -->
+	<!-- Add the Xtion to the arm: code from here https://github.com/JenniferBuehler/common-sensors.git
 	<joint name="toxtion_base" type="fixed">
-        <origin xyz="0 -0.89 -0.01" rpy="0 0 0" />
-        <parent link="tabletop_corner" />
+        <origin xyz="0 0 0" rpy="0 0 0" />
+        <parent link="j2n6s300_link_6" />
         <child link="xtion_base" />
     </joint>
@@ -59,5 +59,5 @@
     <xacro:include filename="$(find common_sensors)/urdf/sensors/xtion.urdf.xacro"/>>
     <xacro:sensor_xtion parent="xtion_base" camera_name="xtion">
-		<origin xyz="0 0 1" rpy="0 -1.57079632679 -1.57079632679" />
-	</xacro:sensor_xtion>
+		<origin xyz="0 -0.08 -0.05" rpy="${J_PI} ${J_PI/2} ${J_PI/2}" />
+	</xacro:sensor_xtion> -->
 </robot>

Commit message: added test for calibration trajectory

File: kinova_description/urdf/arm_on_table.xacro (robot description, xacro)
@@ -14,5 +14,5 @@
 	<xacro:include filename="$(find kinova_description)/urdf/objects/table.xacro" />
 	<joint name="table_to_arm" type="fixed">
-		<origin xyz="0.40488474042 0.27988474042 0.3" rpy="0 0 -${J_PI/4}" />
+		<origin xyz="0.40488474042 0.27988474042 0.3" rpy="0 0 ${J_PI/4}" />
 		<parent link="robot_base"/>
 		<child link="table_base"/>
@@ -49,7 +49,20 @@
 	<xacro:j2n6s300 base_parent="${robot_root}"/>
 	<!-- Add the Xtion to the arm: code from here https://github.com/JenniferBuehler/common-sensors.git
+	<joint name="toxtion_on_arm_base" type="fixed">
+        <origin xyz="0 0 0" rpy="0 0 0" />
+        <parent link="j2n6s300_link_6" />
+        <child link="xtion_on_arm_base" />
+    </joint>
+    <link name="xtion_on_arm_base">
+        <static>false</static>
+    </link>
+    <xacro:include filename="$(find common_sensors)/urdf/sensors/xtion.urdf.xacro"/>>
+    <xacro:sensor_xtion parent="xtion_on_arm_base" camera_name="xtion">
+		<origin xyz="0 -0.08 -0.05" rpy="${J_PI} ${J_PI/2} ${J_PI/2}" />
+	</xacro:sensor_xtion>  -->
+	<!-- Add the Xtion to the world: code from here https://github.com/JenniferBuehler/common-sensors.git -->
 	<joint name="toxtion_base" type="fixed">
         <origin xyz="0 0 0" rpy="0 0 0" />
-        <parent link="j2n6s300_link_6" />
+        <parent link="world" />
         <child link="xtion_base" />
     </joint>
@@ -59,5 +72,5 @@
     <xacro:include filename="$(find common_sensors)/urdf/sensors/xtion.urdf.xacro"/>>
     <xacro:sensor_xtion parent="xtion_base" camera_name="xtion">
-		<origin xyz="0 -0.08 -0.05" rpy="${J_PI} ${J_PI/2} ${J_PI/2}" />
-	</xacro:sensor_xtion> -->
+		<origin xyz="0.5 -1 2" rpy="0 ${J_PI/6} ${J_PI/2}" />
+	</xacro:sensor_xtion>
 </robot>

Commit message: path attempt for calibration

File: kinova_description/urdf/arm_on_table.xacro (robot description, xacro)
@@ -72,5 +72,5 @@
     <xacro:include filename="$(find common_sensors)/urdf/sensors/xtion.urdf.xacro"/>>
     <xacro:sensor_xtion parent="xtion_base" camera_name="xtion">
-		<origin xyz="0.5 -1 2" rpy="0 ${J_PI/6} ${J_PI/2}" />
+		<origin xyz="0.5 -1 1.5" rpy="0 ${J_PI/6} ${J_PI/2}" />
 	</xacro:sensor_xtion>
 </robot>

Commit message: added marker

File: kinova_description/urdf/arm_on_table.xacro (robot description, xacro)
@@ -72,5 +72,13 @@
     <xacro:include filename="$(find common_sensors)/urdf/sensors/xtion.urdf.xacro"/>>
     <xacro:sensor_xtion parent="xtion_base" camera_name="xtion">
-		<origin xyz="0.5 -1 1.5" rpy="0 ${J_PI/6} ${J_PI/2}" />
+		<origin xyz="0.5 -0.8 1.5" rpy="0 ${J_PI/8} ${J_PI/2}" />
 	</xacro:sensor_xtion>
+	<!-- Adding marker -->
+	<joint name="to_marker" type="fixed">
+		<origin xyz="-0.0255 0 -0.12" rpy="0 ${J_PI/2} 0" />
+        <parent link="j2n6s300_link_6" />
+        <child link="marker_4x4_98" />
+    </joint>
+	<xacro:include filename="$(find kinova_description)/urdf/markers/marker_4x4_98.xacro" />
+	<xacro:marker_4x4_98_link link_name="marker_4x4_98"/>
 </robot>

Commit message: added random poses

File: kinova_description/urdf/arm_on_table.xacro (robot description, xacro)
@@ -14,5 +14,5 @@
 	<xacro:include filename="$(find kinova_description)/urdf/objects/table.xacro" />
 	<joint name="table_to_arm" type="fixed">
-		<origin xyz="0.40488474042 0.27988474042 0.3" rpy="0 0 ${J_PI/4}" />
+		<origin xyz="0 0 0.3" rpy="0 0 0" />
 		<parent link="robot_base"/>
 		<child link="table_base"/>
@@ -72,5 +72,5 @@
     <xacro:include filename="$(find common_sensors)/urdf/sensors/xtion.urdf.xacro"/>>
     <xacro:sensor_xtion parent="xtion_base" camera_name="xtion">
-		<origin xyz="0.5 -0.8 1.5" rpy="0 ${J_PI/8} ${J_PI/2}" />
+		<origin xyz="0.5 0.5 3" rpy="0 ${J_PI/2} ${J_PI/2}" />
 	</xacro:sensor_xtion>
 	<!-- Adding marker -->
